File: production/ecad/BMS/power_sheet.kicad_sch (KiCad schematic)
At the start: 4 parts, among them U1 TPS56339DDCR

Commit message: Added heirarchical sheets to main
Parts:
- removed C1, C2: C_Polarized_Small_US, symbol Device:C_Polarized_Small_US
- removed L1: L, symbol Device:L
- removed U1: TPS56339DDCR, TPS56339DDCR:SOT95P280X110-6N, symbol TPS56339DDCR:TPS56339DDCR
