File: production/ecad/BMS/BMS.kicad_sch (KiCad schematic)
At the start: 7 parts, among them J7 ADC-028-1-T/R-PA10T, U3 TPS75233QPWPREP

Commit message: Barrel jack updated
Other:
- note added: "Barrel jack connector: 5V from wall adapter"
- moved on the sheet: J7
Changed lines of the file:
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@@
 	(wire
 		(pts
-			(xy 238.76 49.53) (xy 251.46 49.53)
+			(xy 226.06 45.72) (xy 238.76 45.72)
 		)
 		(stroke
@@
 	(wire
 		(pts
-			(xy 238.76 41.91) (xy 251.46 41.91)
+			(xy 226.06 38.1) (xy 238.76 38.1)
 		)
 		(stroke
@@
 			(width 0)
 			(type default)
+		)
+	)
+	(rectangle
+		(start 176.53 16.51)
+		(end 283.21 55.88)
+		(stroke
+			(width 1)
+			(type default)
+		)
+		(fill
+			(type none)
 		)
 	)
@@
 		)
 	)
+	(text "Barrel jack connector: 5V from wall adapter"
+		(exclude_from_sim no)
+		(at 178.308 24.638 0)
+		(effects
+			(font
+				(size 3 3)
+				(thickness 0.6)
+				(bold yes)
+			)
+			(justify left bottom)
+		)
+	)
 	(text "LDO: 5V to 3.3V, 2A\n\n"
 		(exclude_from_sim no)
@@
 	(hierarchical_label "5VEXT"
 		(shape input)
-		(at 251.46 49.53 0)
+		(at 238.76 45.72 0)
 		(fields_autoplaced yes)
 		(effects
@@
 	(hierarchical_label "GND"
 		(shape input)
-		(at 251.46 41.91 0)
+		(at 238.76 38.1 0)
 		(fields_autoplaced yes)
 		(effects
@@
 	(symbol
 		(lib_id "2024-10-20_20-22-38:ADC-028-1-T_R-PA10T")
-		(at 238.76 41.91 0)
+		(at 226.06 38.1 0)
 		(unit 1)
 		(exclude_from_sim no)
@@
 		(fields_autoplaced yes)
 		(property "Reference" "J7"
-			(at 225.4278 36.83 0)
+			(at 212.7278 33.02 0)
 			(effects
 				(font
@@
 		)
 		(property "Value" "ADC-028-1-T/R-PA10T"
-			(at 225.4278 39.37 0)
+			(at 212.7278 35.56 0)
 			(effects
 				(font
@@
 		)
 		(property "Footprint" "ADC-028-x-T/R-PA10T_ADM"
-			(at 238.76 41.91 0)
+			(at 226.06 38.1 0)
 			(effects
 				(font
@@
 		)
 		(property "Datasheet" "ADC-028-1-T/R-PA10T"
-			(at 238.76 41.91 0)
+			(at 226.06 38.1 0)
 			(effects
 				(font
@@
 		)
 		(property "Description" ""
-			(at 238.76 41.91 0)
+			(at 226.06 38.1 0)
 			(effects
 				(font
