File: production/ecad/Peripheral/Peripheral.kicad_sch (KiCad schematic)
At the start: 1 part, among them J2 214721-0100

Commit message: hierachel stuff
Connections:
- net SW1: now reaches J2.3
- net SW2: now reaches J2.4
- net SW3: now reaches J2.5
- net SW4: now reaches J2.6
- net SW5: now reaches J2.7
- net COMA: now reaches J2.8
- net COMB: now reaches J2.9
- no-connect marks 0 -> 1
Changed lines of the file:
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@@
 	(generator_version "8.0")
 	(paper "A4")
+	(no_connect
+		(at 119.38 91.44)
+	)
+	(hierarchical_label "SW1"
+		(shape input)
+		(at 119.38 73.66 0)
+		(fields_autoplaced yes)
+		(effects
+			(font
+				(size 1.27 1.27)
+			)
+			(justify left)
+		)
+	)
+	(hierarchical_label "COMB"
+		(shape input)
+		(at 119.38 88.9 0)
+		(fields_autoplaced yes)
+		(effects
+			(font
+				(size 1.27 1.27)
+			)
+			(justify left)
+		)
+	)
 	(hierarchical_label "ENCA"
 		(shape input)
 		(at 119.38 68.58 0)
+		(fields_autoplaced yes)
+		(effects
+			(font
+				(size 1.27 1.27)
+			)
+			(justify left)
+		)
+	)
+	(hierarchical_label "SW3"
+		(shape input)
+		(at 119.38 78.74 0)
 		(fields_autoplaced yes)
 		(effects
@@
 		(fields_autoplaced yes)
 		(effects
+			(font
+				(size 1.27 1.27)
+			)
+			(justify left)
+		)
+	)
+	(hierarchical_label "SW2"
+		(shape input)
+		(at 119.38 76.2 0)
+		(fields_autoplaced yes)
+		(effects
+			(font
+				(size 1.27 1.27)
+			)
+			(justify left)
+		)
+	)
+	(hierarchical_label "SW5"
+		(shape input)
+		(at 119.38 83.82 0)
+		(fields_autoplaced yes)
+		(effects
+			(font
+				(size 1.27 1.27)
+			)
+			(justify left)
+		)
+	)
+	(hierarchical_label "COMA"
+		(shape input)
+		(at 119.38 86.36 0)
+		(fields_autoplaced yes)
+		(effects
+			(font
+				(size 1.27 1.27)
+			)
+			(justify left)
+		)
+	)
+	(hierarchical_label "SW4"
+		(shape input)
+		(at 119.38 81.28 0)
+		(fields_autoplaced yes)
+		(effects
