File: production/ecad/Peripheral/Peripheral.kicad_sch (KiCad schematic)
At the start: 1 part, among them J2 214721-0100

Commit message: updated schem
Connections:
- net COMA renamed ANO_COMA
- net COMB renamed ANO_COMB
- net ENCA renamed ANO_ENCA
- net ENCB renamed ANO_ENCB
- net SW1 renamed ANO_SW1
- net SW2 renamed ANO_SW2
- net SW3 renamed ANO_SW3
- net SW4 renamed ANO_SW4
- net SW5 renamed ANO_SW5
Changed lines of the file:
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@@
 		(at 93.98 71.12)
 	)
-	(hierarchical_label "SW1"
+	(hierarchical_label "ANO_SW1"
 		(shape input)
 		(at 119.38 73.66 0)
@@
 		)
 	)
-	(hierarchical_label "COMB"
+	(hierarchical_label "ANO_COMB"
 		(shape input)
 		(at 119.38 88.9 0)
@@
 		)
 	)
-	(hierarchical_label "ENCA"
+	(hierarchical_label "ANO_ENCA"
 		(shape input)
 		(at 119.38 68.58 0)
@@
 		)
 	)
-	(hierarchical_label "SW3"
+	(hierarchical_label "ANO_SW3"
 		(shape input)
 		(at 119.38 78.74 0)
@@
 		)
 	)
-	(hierarchical_label "ENCB"
+	(hierarchical_label "ANO_ENCB"
 		(shape input)
 		(at 119.38 71.12 0)
@@
 		)
 	)
-	(hierarchical_label "SW2"
+	(hierarchical_label "ANO_SW2"
 		(shape input)
 		(at 119.38 76.2 0)
@@
 		)
 	)
-	(hierarchical_label "SW5"
+	(hierarchical_label "ANO_SW5"
 		(shape input)
 		(at 119.38 83.82 0)
@@
 		)
 	)
-	(hierarchical_label "COMA"
+	(hierarchical_label "ANO_COMA"
 		(shape input)
 		(at 119.38 86.36 0)
@@
 		)
 	)
-	(hierarchical_label "SW4"
+	(hierarchical_label "ANO_SW4"
 		(shape input)
 		(at 119.38 81.28 0)
