File: production/ecad/Motor/Motor.kicad_sch (KiCad schematic)
At the start: 0 parts

Commit message: added motor/LCD
Parts:
- added J4, J5, J6: 214721-0020, 2147210020, symbol 2positionheader:214721-0020
- added Q1, Q2: NMOS, symbol Simulation_SPICE:NMOS
- added U1: DRV8871DDA, Package_SO:Texas_HTSOP-8-1EP_3.9x4.9mm_P1.27mm_EP2.95x4.9mm_Mask2.4x3.1mm_ThermalVias, symbol Driver_Motor:DRV8871DDA
Connections:
- new net: J5.2, Q2.3 (S)
- new net: J6.2, U1.6 (OUT1)
- new net: J6.1, U1.8 (OUT2)
- new net: J4.2, Q1.3 (S)
- new net 3.3VEXT: Q1.1 (D), Q2.1 (D)
- new net 6.5VEXT: U1.4 (ILIM)
- new net GNDEXT: J4.1, J5.1, U1.1 (GND), U1.7 (GND), U1.9 (GND)
- new net MTR_IN1: U1.3 (IN1)
- new net MTR_IN2: U1.2 (IN2)
- new net VBR_MTR_EN1: Q1.2 (G)
- new net VBR_MTR_EN2: Q2.2 (G)
- no-connect marks 0 -> 6
Other:
- note added: "IF NOT, BACK UP MOTOR DRIVER IS TB6612"
- note added: "MOTOR DRIVER NEEDS 6.5V, BUT MOTOR NEEDS 6V. CONFLICT?"
- note added: "https://www.sparkfun.com/products/14451"

Commit message: updated schem
Parts:
- added R1: R_US, symbol Device:R_US
Connections:
- net 5VEXT: now reaches U1.5 (VM)
- net 6.5VEXT: no longer names the net of U1.4 (ILIM)
- net 6.5VEXT: now also R1.1
- new net GND: R1.2
Other:
- note added: "MOTOR DRIVER NEEDS 6.5V, BUT MOTOR NEEDS 5V. SHOULD WE CHANGE MOTOR DRIVER TO BELOW?"
- note removed: "MOTOR DRIVER NEEDS 6.5V, BUT MOTOR NEEDS 6V. CONFLICT?"
Changed lines of the file:
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@@
 		)
 	)
-	(text "MOTOR DRIVER NEEDS 6.5V, BUT MOTOR NEEDS 6V. CONFLICT?"
+	(text "MOTOR DRIVER NEEDS 6.5V, BUT MOTOR NEEDS 5V. SHOULD WE CHANGE MOTOR DRIVER TO BELOW?"
 		(exclude_from_sim no)
 		(at 131.572 95.504 0)
@@
 		)
 	)
+	(label "CURRENT LIM RES"
+		(at 125.73 85.09 0)
+		(fields_autoplaced yes)
+		(effects
+			(font
+				(size 1.27 1.27)
+			)
+			(justify left bottom)
+		)
+	)
 	(hierarchical_label "VBR_MTR_EN1"
 		(shape input)
@@
 		)
 	)
+	(hierarchical_label "5VEXT"
+		(shape input)
+		(at 115.57 68.58 0)
+		(fields_autoplaced yes)
+		(effects
+			(font
+				(size 1.27 1.27)
+			)
+			(justify left)
+		)
+	)
 	(hierarchical_label "GNDEXT"
 		(shape input)
@@
 			)
 			(justify right)
-		)
-	)
-	(hierarchical_label "6.5VEXT"
-		(shape input)
-		(at 125.73 81.28 0)
-		(fields_autoplaced yes)
-		(effects
-			(font
-				(size 1.27 1.27)
-			)
-			(justify left)
 		)
 	)
@@
 					(unit 1)
 				)
+			)
+		)
+	)
+	(symbol
+		(lib_id "power:GND")
+		(at 133.35 81.28 0)
+		(unit 1)
+		(exclude_from_sim no)
+		(in_bom yes)
+		(on_board yes)
+		(dnp no)
+		(fields_autoplaced yes)
+		(property "Reference" "#PWR01"
+			(at 133.35 87.63 0)
+			(effects
+				(font
+					(size 1.27 1.27)
+				)
+				(hide yes)
+			)
+		)
+		(property "Value" "GND"
+			(at 133.35 86.36 0)
+			(effects
+				(font
+					(size 1.27 1.27)
+				)
+			)
+		)
+		(property "Footprint" ""
+			(at 133.35 81.28 0)
+			(effects
+				(font
+					(size 1.27 1.27)
+				)
+				(hide yes)
+			)
+		)
+		(property "Datasheet" ""
+			(at 133.35 81.28 0)
+			(effects
+				(font
+					(size 1.27 1.27)
+				)
+				(hide yes)
+			)
+		)
+		(property "Description" "Power symbol creates a global label with name \"GND\" , ground"
+			(at 133.35 81.28 0)
+			(effects
+				(font
+					(size 1.27 1.27)
+				)
+				(hide yes)
+			)
+		)
+		(pin "1"
+		)
+		(instances
+			(project ""
+				(path "/a34d77bc-8f6a-417e-a206-3165e6c5c658/682b5c07-6a85-4a0a-86de-ba40b1ceb9db"
+					(reference "#PWR01")
+					(unit 1)
+				)
+			)
+		)
+	)
+	(symbol
+		(lib_id "Device:R_US")
+		(at 129.54 81.28 90)
+		(unit 1)
+		(exclude_from_sim no)
+		(in_bom yes)
+		(on_board yes)
+		(dnp no)
+		(fields_autoplaced yes)
+		(property "Reference" "R1"
+			(at 129.54 74.93 90)
+			(effects
+				(font
+					(size 1.27 1.27)
+				)
+			)
+		)
+		(property "Value" "R_US"
+			(at 129.54 77.47 90)
+			(effects
+				(font
+					(size 1.27 1.27)
+				)
+			)
+		)
+		(property "Footprint" ""
+			(at 129.794 80.264 90)
+			(effects
+				(font
+					(size 1.27 1.27)
+				)
+				(hide yes)
+			)
+		)
+		(property "Datasheet" "~"
+			(at 129.54 81.28 0)
+			(effects
+				(font
+					(size 1.27 1.27)
+				)
+				(hide yes)
+			)
+		)
+		(property "Description" "Resistor, US symbol"
+			(at 129.54 81.28 0)
+			(effects
+				(font
+					(size 1.27 1.27)
+				)
+				(hide yes)
+			)
+		)
+		(pin "1"
+		)
+		(pin "2"
+		)
+		(instances
+			(project ""
+				(path "/a34d77bc-8f6a-417e-a206-3165e6c5c658/682b5c07-6a85-4a0a-86de-ba40b1ceb9db"
+					(reference "R1")
+					(unit 1)
+				)

Commit message: schematic draft merged w neha
Parts:
- removed R1: R_US, symbol Device:R_US
- removed U1: DRV8871DDA, Package_SO:Texas_HTSOP-8-1EP_3.9x4.9mm_P1.27mm_EP2.95x4.9mm_Mask2.4x3.1mm_ThermalVias, symbol Driver_Motor:DRV8871DDA
- added U1: TB6612FNG, Package_SO:SSOP-24_5.3x8.2mm_P0.65mm, symbol Driver_Motor:TB6612FNG
Connections:
- net 5VEXT: now also U1.20 (VCC), U1.24 (VM1)
- net GNDEXT: now also U1.18 (GND)
- net MTR_IN1: now also U1.23 (PWMA)
- net at J6.2: now also U1.1 (AO1), U1.2 (AO1)
- net at J6.1: now also U1.5 (AO2), U1.6 (AO2)
- net 3.3VEXT renamed 3V3EXT
- new net: U1.10 (PGND2), U1.9 (PGND2)
- new net: U1.11 (BO1), U1.12 (BO1)
- new net: U1.3 (PGND1), U1.4 (PGND1)
- new net: U1.7 (BO2), U1.8 (BO2)
- new net MTR_DIR1: U1.21 (AIN1)
- new net MTR_DIR2: U1.22 (AIN2)
- new net MTR_EN1: U1.19 (STBY)
- no-connect marks 6 -> 15
Other:
- note removed: "IF NOT, BACK UP MOTOR DRIVER IS TB6612"
- note removed: "MOTOR DRIVER NEEDS 6.5V, BUT MOTOR NEEDS 5V. SHOULD WE CHANGE MOTOR DRIVER TO BELOW?"
- note removed: "https://www.sparkfun.com/products/14451"
