File: production/ecad/Motor/Motor.kicad_sch (KiCad schematic)
At the start: 6 parts, among them J4 214721-0020, J5 214721-0020, J6 214721-0020, Q1 NMOS, Q2 NMOS, U1 TB6612FNG

Commit message: schematic changes and pcb
Connections:
- net GND: now also J4.MP1, J4.MP2, J5.MP1, J5.MP2, J6.MP1, J6.MP2
- no-connect marks 13 -> 7

Commit message: changed fet footp
Parts:
- Q1, Q2: footprint Transistor_Power:GaN_Systems_GaNPX-3_5x6.6mm_Drain3.76x0.6mm -> Footprints:SOT50P160X90-3N
Changed lines of the file:
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@@
 			)
 		)
-		(property "Footprint" "Transistor_Power:GaN_Systems_GaNPX-3_5x6.6mm_Drain3.76x0.6mm"
+		(property "Footprint" "Footprints:SOT50P160X90-3N"
 			(at 55.88 71.12 0)
 			(effects
@@
 			)
 		)
-		(property "Footprint" "Transistor_Power:GaN_Systems_GaNPX-3_5x6.6mm_Drain3.76x0.6mm"
+		(property "Footprint" "Footprints:SOT50P160X90-3N"
 			(at 55.88 36.83 0)
 			(effects
