File: production/ecad/ANO-DIAL/ANO-DIAL.kicad_sch (KiCad schematic)
At the start: 1 part, among them J2 214721-0100

Commit message: merged with main
Parts:
- J2: footprint 2147210100 -> footprints:10positionheader
Changed lines of the file:
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@@
 			)
 		)
-		(property "Footprint" "2147210100"
+		(property "Footprint" "footprints:10positionheader"
 			(at 115.57 163.5 0)
 			(effects
