File: production/ecad/ANO-DIAL/ANO-DIAL.kicad_sch (KiCad schematic)
At the start: 1 part, among them J2 214721-0100

Commit message: connectors
Parts:
- J2: footprint 2147210100 -> Fitolux:8positionheader
Changed lines of the file:
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@@
 			)
 		)
-		(property "Footprint" "2147210100"
+		(property "Footprint" "Fitolux:8positionheader"
 			(at 115.57 163.5 0)
 			(effects

Commit message: Component placement complete
Parts:
- J2: footprint Fitolux:8positionheader -> Footprints:8positionheader
Changed lines of the file:
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@@
 			)
 		)
-		(property "Footprint" "Fitolux:8positionheader"
+		(property "Footprint" "Footprints:8positionheader"
 			(at 115.57 163.5 0)
 			(effects

Commit message: schematic changes and pcb
Parts:
- added R10, R11, R12, R13, R9: 4.7k, Resistor_SMD:R_0201_0603Metric, symbol Device:R
Connections:
- net ANO_SW1: now also R9.2
- net ANO_SW2: now also R10.2
- net ANO_SW3: now also R11.2
- net ANO_SW4: now also R12.2
- net ANO_SW5: now also R13.2
- net GND: now reaches J2.MP1
- net GND: now also J2.MP2
- new net 3V3EXT: R10.1, R11.1, R12.1, R13.1, R9.1
- no-connect marks 3 -> 1

Commit message: resistor and inductor
Parts:
- R10, R11, R12, R13, R9: footprint Resistor_SMD:R_0201_0603Metric -> Resistor_SMD:R_0603_1608Metric
Changed lines of the file:
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@@
 			)
 		)
-		(property "Footprint" "Resistor_SMD:R_0201_0603Metric"
+		(property "Footprint" "Resistor_SMD:R_0603_1608Metric"
 			(at 146.812 104.14 90)
 			(effects
@@
 			)
 		)
-		(property "Footprint" "Resistor_SMD:R_0201_0603Metric"
+		(property "Footprint" "Resistor_SMD:R_0603_1608Metric"
 			(at 148.082 120.65 90)
 			(effects
@@
 			)
 		)
-		(property "Footprint" "Resistor_SMD:R_0201_0603Metric"
+		(property "Footprint" "Resistor_SMD:R_0603_1608Metric"
 			(at 149.352 87.63 90)
 			(effects
@@
 			)
 		)
-		(property "Footprint" "Resistor_SMD:R_0201_0603Metric"
+		(property "Footprint" "Resistor_SMD:R_0603_1608Metric"
 			(at 146.812 142.24 90)
 			(effects
@@
 			)
 		)
-		(property "Footprint" "Resistor_SMD:R_0201_0603Metric"
+		(property "Footprint" "Resistor_SMD:R_0603_1608Metric"
 			(at 149.352 73.66 90)
 			(effects
