File: production/ecad/IMU/IMU.kicad_sch (KiCad schematic)
At the start: 1 part, among them J1 214721-0061

Commit message: merged with main
Parts:
- J1: footprint 2147210061 -> footprints:6_pos_connector
Changed lines of the file:
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@@
 			)
 		)
-		(property "Footprint" "2147210061"
+		(property "Footprint" "footprints:6_pos_connector"
 			(at 132.08 190.17 0)
 			(effects
