File: production/ecad/IMU/IMU.kicad_sch (KiCad schematic)
At the start: 1 part, among them J1 214721-0061

Commit message: connectors
Parts:
- J1: footprint 2147210061 -> Fitolux:6_pos_connector
Changed lines of the file:
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@@
 			)
 		)
-		(property "Footprint" "2147210061"
+		(property "Footprint" "Fitolux:6_pos_connector"
 			(at 132.08 190.17 0)
 			(effects

Commit message: Component placement complete
Parts:
- J1: footprint Fitolux:6_pos_connector -> Footprints:6_pos_connector
Changed lines of the file:
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@@
 			)
 		)
-		(property "Footprint" "Fitolux:6_pos_connector"
+		(property "Footprint" "Footprints:6_pos_connector"
 			(at 132.08 190.17 0)
 			(effects

Commit message: schematic changes and pcb
Connections:
- net GND: now reaches J1.7 (MP1)
- net GND: now also J1.8 (MP2)
- no-connect marks 3 -> 1
Changed lines of the file:
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@@
 	(paper "A4")
-	(no_connect
-		(at 113.03 97.79)
-	)
-	(no_connect
-		(at 113.03 95.25)
-	)
 	(no_connect
 		(at 135.89 95.25)
@@
 					(unit 1)
 				)
+			)
+		)
+	)
+	(symbol
+		(lib_id "power:GND")
+		(at 113.03 97.79 270)
+		(unit 1)
+		(exclude_from_sim no)
+		(in_bom yes)
+		(on_board yes)
+		(dnp no)
+		(property "Reference" "#PWR059"
+			(at 106.68 97.79 0)
+			(effects
+				(font
+					(size 1.27 1.27)
+				)
+				(hide yes)
+			)
+		)
+		(property "Value" "GND"
+			(at 109.22 97.7901 90)
+			(effects
+				(font
+					(size 1.27 1.27)
+				)
+				(justify right)
+			)
+		)
+		(property "Footprint" ""
+			(at 113.03 97.79 0)
+			(effects
+				(font
+					(size 1.27 1.27)
+				)
+				(hide yes)
+			)
+		)
+		(property "Datasheet" ""
+			(at 113.03 97.79 0)
+			(effects
+				(font
+					(size 1.27 1.27)
+				)
+				(hide yes)
+			)
+		)
+		(property "Description" "Power symbol creates a global label with name \"GND\" , ground"
+			(at 113.03 97.79 0)
+			(effects
+				(font
+					(size 1.27 1.27)
+				)
+				(hide yes)
+			)
+		)
+		(pin "1"
+		)
+		(instances
+			(project "Main"
+				(path "/a34d77bc-8f6a-417e-a206-3165e6c5c658/2c3b99aa-7fc3-47b6-80fb-b33e75ed001e"
+					(reference "#PWR059")
+					(unit 1)
+				)
+			)
+		)
+	)
+	(symbol
+		(lib_id "power:GND")
+		(at 113.03 95.25 270)
+		(unit 1)
+		(exclude_from_sim no)
+		(in_bom yes)
+		(on_board yes)
+		(dnp no)
+		(property "Reference" "#PWR058"
+			(at 106.68 95.25 0)
+			(effects
+				(font
+					(size 1.27 1.27)
+				)
+				(hide yes)
+			)
+		)
+		(property "Value" "GND"
+			(at 109.22 95.2501 90)
+			(effects
+				(font
+					(size 1.27 1.27)
+				)
+				(justify right)
+			)
+		)
+		(property "Footprint" ""
+			(at 113.03 95.25 0)
+			(effects
+				(font
+					(size 1.27 1.27)
+				)
+				(hide yes)
+			)
+		)
+		(property "Datasheet" ""
+			(at 113.03 95.25 0)
+			(effects
+				(font
+					(size 1.27 1.27)
+				)
+				(hide yes)
+			)
+		)
+		(property "Description" "Power symbol creates a global label with name \"GND\" , ground"
+			(at 113.03 95.25 0)
+			(effects
+				(font
+					(size 1.27 1.27)
+				)
+				(hide yes)
+			)
+		)
+		(pin "1"
+		)
+		(instances
+			(project "Main"
+				(path "/a34d77bc-8f6a-417e-a206-3165e6c5c658/2c3b99aa-7fc3-47b6-80fb-b33e75ed001e"
+					(reference "#PWR058")
+					(unit 1)
+				)
