File: production/ecad/LOAD-CELL/LOAD-CELL.kicad_sch (KiCad schematic)
At the start: 17 parts, among them J10 214721-0061, Q3 MMBT4403, U3 HX711

Commit message: Stylistic edits made
Parts:
- removed SJ1: JUMPER-PAD-2-NC_BY_TRACE, Load Cell and Amplifier:PAD-JUMPER-2-NC_BY_TRACE_YES_SILK, symbol Load Cell and Amplifier-eagle-import:JUMPER-PAD-2-NC_BY_TRACE
- added DNP1: 0, symbol Device:R
Connections:
- net VDD is gone; now on net +5V: C4.1, U3.16 (DVDD)
- net GND: now also DNP1.1
- net at R7.1, U3.15 (RATE): now also DNP1.2
- net VCC renamed +5V
Other:
- moved on the sheet: C4, C6, C7

Commit message: more changes
Connections:
- no-connect marks 5 -> 6
Changed lines of the file:
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@@
+	)
+	(no_connect
+		(at 190.5 86.36)
 	)
 	(no_connect
@@
 	(wire
 		(pts
-			(xy 190.5 91.44) (xy 237.49 91.44)
-		)
-		(stroke
-			(width 0.1524)
-			(type solid)
-		)
-	)
-	(wire
-		(pts
-			(xy 190.5 96.52) (xy 195.58 96.52)
+			(xy 190.5 91.44) (xy 210.82 91.44)
+		)
+		(stroke
+			(width 0.1524)
+			(type solid)
+		)
+	)
+	(wire
+		(pts
+			(xy 190.5 96.52) (xy 210.82 96.52)
 		)
 		(stroke
@@
 		(pts
 			(xy 157.48 63.5) (xy 157.48 76.2)
-		)
-		(stroke
-			(width 0.1524)
-			(type solid)
-		)
-	)
-	(wire
-		(pts
-			(xy 195.58 93.98) (xy 237.49 93.98)
 		)
 		(stroke
@@
 		(pts
 			(xy 88.9 124.46) (xy 88.9 78.74)
-		)
-		(stroke
-			(width 0.1524)
-			(type solid)
-		)
-	)
-	(wire
-		(pts
-			(xy 195.58 96.52) (xy 195.58 93.98)
 		)
 		(stroke
@@
 		)
 	)
-	(label "SCK"
-		(at 215.9 93.98 0)
-		(fields_autoplaced yes)
-		(effects
-			(font
-				(size 1.2446 1.2446)
-			)
-			(justify left bottom)
-		)
-	)
-	(label "DAT"
-		(at 215.9 91.44 0)
-		(fields_autoplaced yes)
-		(effects
-			(font
-				(size 1.2446 1.2446)
-			)
-			(justify left bottom)
-		)
-	)
 	(label "A+"
 		(at 81.28 78.74 0)
@@
 	(hierarchical_label "DAT"
 		(shape output)
-		(at 237.49 91.44 0)
+		(at 210.82 91.44 0)
 		(fields_autoplaced yes)
 		(effects
@@
 	(hierarchical_label "SCK"
 		(shape output)
-		(at 237.49 93.98 0)
+		(at 210.82 96.52 0)
 		(fields_autoplaced yes)
 		(effects

Commit message: added some footprints
Parts:
- J10: footprint 2147210061 -> LoadCellFootprints:6_pos_connector
- U3: footprint Load Cell and Amplifier:SO16 -> LoadCellFootprints:HX711
Changed lines of the file:
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@@
 			)
 		)
-		(property "Footprint" "Load Cell and Amplifier:SO16"
+		(property "Footprint" "LoadCellFootprints:HX711"
 			(at 177.8 88.9 0)
 			(effects
@@
 			)
 		)
-		(property "Footprint" "2147210061"
+		(property "Footprint" "LoadCellFootprints:6_pos_connector"
 			(at 72.39 166.04 0)
 			(effects

Commit message: Added more footprints
Parts:
- C3, C4, C6, C8, C9: footprint Load Cell and Amplifier:0603-CAP -> LoadCellFootprints:0p1uF
- C5, C7: footprint Load Cell and Amplifier:1210 -> LoadCellFootprints:10uF
- DNP1: footprint (none) -> LoadCellFootprints:10k
- L1: footprint Load Cell and Amplifier:0805 -> LoadCellFootprints:inductor
- Q3: footprint Load Cell and Amplifier:SOT23-3 -> LoadCellFootprints:mmbt4403
- R3: footprint Load Cell and Amplifier:0603-RES -> LoadCellFootprints:20k
- R4: footprint Load Cell and Amplifier:0603-RES -> LoadCellFootprints:8p2k
- R5, R6: footprint Load Cell and Amplifier:0603-RES -> LoadCellFootprints:100ohm
- R7: footprint Load Cell and Amplifier:0603-RES -> LoadCellFootprints:10k
Changed lines of the file:
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@@
 			)
 		)
-		(property "Footprint" ""
+		(property "Footprint" "LoadCellFootprints:10k"
 			(at 204.978 74.93 90)
 			(effects
@@
 			)
 		)
-		(property "Footprint" "Load Cell and Amplifier:0603-RES"
+		(property "Footprint" "LoadCellFootprints:100ohm"
 			(at 139.7 111.76 0)
 			(effects
@@
 			)
 		)
-		(property "Footprint" "Load Cell and Amplifier:1210"
+		(property "Footprint" "LoadCellFootprints:10uF"
 			(at 109.22 78.74 0)
 			(effects
@@
 			)
 		)
-		(property "Footprint" "Load Cell and Amplifier:0805"
+		(property "Footprint" "LoadCellFootprints:inductor"
 			(at 124.46 71.12 0)
 			(effects
@@
 			)
 		)
-		(property "Footprint" "Load Cell and Amplifier:0603-RES"
+		(property "Footprint" "LoadCellFootprints:100ohm"
 			(at 139.7 124.46 0)
 			(effects
@@
 			)
 		)
-		(property "Footprint" "Load Cell and Amplifier:0603-CAP"
+		(property "Footprint" "LoadCellFootprints:0p1uF"
 			(at 149.86 101.6 0)
 			(effects
@@
 			)
 		)
-		(property "Footprint" "Load Cell and Amplifier:0603-CAP"
+		(property "Footprint" "LoadCellFootprints:0p1uF"
 			(at 92.71 31.75 0)
 			(effects
@@
 			)
 		)
-		(property "Footprint" "Load Cell and Amplifier:0603-CAP"
+		(property "Footprint" "LoadCellFootprints:0p1uF"
 			(at 147.32 119.38 0)
 			(effects
@@
 			)
 		)
-		(property "Footprint" "Load Cell and Amplifier:0603-RES"
+		(property "Footprint" "LoadCellFootprints:8p2k"
 			(at 137.16 93.98 0)
 			(effects
@@
 			)
 		)
-		(property "Footprint" "Load Cell and Amplifier:SOT23-3"
+		(property "Footprint" "LoadCellFootprints:mmbt4403"
 			(at 144.78 63.5 0)
 			(effects
@@
 			)
 		)
-		(property "Footprint" "Load Cell and Amplifier:0603-CAP"
+		(property "Footprint" "LoadCellFootprints:0p1uF"
 			(at 105.41 31.75 0)
 			(effects
@@
 			)
 		)
-		(property "Footprint" "Load Cell and Amplifier:0603-CAP"
+		(property "Footprint" "LoadCellFootprints:0p1uF"
 			(at 99.06 78.74 0)
 			(effects
@@
 			)
 		)
-		(property "Footprint" "Load Cell and Amplifier:0603-RES"
+		(property "Footprint" "LoadCellFootprints:10k"
 			(at 203.2 60.96 0)
 			(effects
@@
 			)
 		)
-		(property "Footprint" "Load Cell and Amplifier:1210"
+		(property "Footprint" "LoadCellFootprints:10uF"
 			(at 120.65 31.75 0)
 			(effects
@@
 			)
 		)
-		(property "Footprint" "Load Cell and Amplifier:0603-RES"
+		(property "Footprint" "LoadCellFootprints:20k"
 			(at 137.16 78.74 0)
 			(effects

Commit message: merged with main
Parts:
- C3, C4, C6, C8, C9: footprint LoadCellFootprints:0p1uF -> Footprints:0p1uF
- C5, C7: footprint LoadCellFootprints:10uF -> Footprints:10uF
- DNP1, R7: footprint LoadCellFootprints:10k -> Footprints:10k
- J10: footprint LoadCellFootprints:6_pos_connector -> Footprints:6_pos_connector
- L1: footprint LoadCellFootprints:inductor -> Footprints:inductor
- Q3: footprint LoadCellFootprints:mmbt4403 -> Footprints:mmbt4403
- R3: footprint LoadCellFootprints:20k -> Footprints:20k
- R4: footprint LoadCellFootprints:8p2k -> Footprints:8p2k
- R5, R6: footprint LoadCellFootprints:100ohm -> Footprints:100ohm
- U3: footprint LoadCellFootprints:HX711 -> Footprints:HX711
Changed lines of the file:
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@@
 			)
 		)
-		(property "Footprint" "LoadCellFootprints:10k"
+		(property "Footprint" "Footprints:10k"
 			(at 204.978 74.93 90)
 			(effects
@@
 			)
 		)
-		(property "Footprint" "LoadCellFootprints:100ohm"
+		(property "Footprint" "Footprints:100ohm"
 			(at 139.7 111.76 0)
 			(effects
@@
 			)
 		)
-		(property "Footprint" "LoadCellFootprints:10uF"
+		(property "Footprint" "Footprints:10uF"
 			(at 109.22 78.74 0)
 			(effects
@@
 			)
 		)
-		(property "Footprint" "LoadCellFootprints:inductor"
+		(property "Footprint" "Footprints:inductor"
 			(at 124.46 71.12 0)
 			(effects
@@
 			)
 		)
-		(property "Footprint" "LoadCellFootprints:HX711"
+		(property "Footprint" "Footprints:HX711"
 			(at 177.8 88.9 0)
 			(effects
@@
 			)
 		)
-		(property "Footprint" "LoadCellFootprints:100ohm"
+		(property "Footprint" "Footprints:100ohm"
 			(at 139.7 124.46 0)
 			(effects
@@
 			)
 		)
-		(property "Footprint" "LoadCellFootprints:0p1uF"
+		(property "Footprint" "Footprints:0p1uF"
 			(at 149.86 101.6 0)
 			(effects
@@
 			)
 		)
-		(property "Footprint" "LoadCellFootprints:0p1uF"
+		(property "Footprint" "Footprints:0p1uF"
 			(at 92.71 31.75 0)
 			(effects
@@
 			)
 		)
-		(property "Footprint" "LoadCellFootprints:0p1uF"
+		(property "Footprint" "Footprints:0p1uF"
 			(at 147.32 119.38 0)
 			(effects
@@
 			)
 		)
-		(property "Footprint" "LoadCellFootprints:8p2k"
+		(property "Footprint" "Footprints:8p2k"
 			(at 137.16 93.98 0)
 			(effects
@@
 			)
 		)
-		(property "Footprint" "LoadCellFootprints:mmbt4403"
+		(property "Footprint" "Footprints:mmbt4403"
 			(at 144.78 63.5 0)
 			(effects
@@
 			)
 		)
-		(property "Footprint" "LoadCellFootprints:6_pos_connector"
+		(property "Footprint" "Footprints:6_pos_connector"
 			(at 72.39 166.04 0)
 			(effects
@@
 			)
 		)
-		(property "Footprint" "LoadCellFootprints:0p1uF"
+		(property "Footprint" "Footprints:0p1uF"
 			(at 105.41 31.75 0)
 			(effects
@@
 			)
 		)
-		(property "Footprint" "LoadCellFootprints:0p1uF"
+		(property "Footprint" "Footprints:0p1uF"
 			(at 99.06 78.74 0)
 			(effects
@@
 			)
 		)
-		(property "Footprint" "LoadCellFootprints:10k"
+		(property "Footprint" "Footprints:10k"
 			(at 203.2 60.96 0)
 			(effects
@@
 			)
 		)
-		(property "Footprint" "LoadCellFootprints:10uF"
+		(property "Footprint" "Footprints:10uF"
 			(at 120.65 31.75 0)
 			(effects
@@
 			)
 		)
-		(property "Footprint" "LoadCellFootprints:20k"
+		(property "Footprint" "Footprints:20k"
 			(at 137.16 78.74 0)
 			(effects
