File: production/ecad/LOAD-CELL/LOAD-CELL.kicad_sch (KiCad schematic)
At the start: 17 parts, among them J10 214721-0061, Q3 MMBT4403, U3 HX711

Commit message: Component placement complete
Parts:
- renumbered DNP1 to DNP3
Changed lines of the file:
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@@
 		(on_board yes)
 		(dnp no)
-		(property "Reference" "DNP1"
+		(property "Reference" "DNP3"
 			(at 205.486 77.216 90)
 			(effects
@@
 			(project "Main"
 				(path "/a34d77bc-8f6a-417e-a206-3165e6c5c658/1fa8e4ec-3b8f-41b7-8956-25ba2b294586"
-					(reference "DNP1")
+					(reference "DNP3")
 					(unit 1)
 				)

Commit message: schematic changes and pcb
Connections:
- net GND: now also J10.6, J10.7 (MP1), J10.8 (MP2)
- no-connect marks 6 -> 3
Changed lines of the file:
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@@
-	)
-	(no_connect
-		(at 53.34 71.12)
-	)
-	(no_connect
-		(at 53.34 73.66)
 	)
 	(no_connect
@@
 	(no_connect
 		(at 190.5 86.36)
-	)
-	(no_connect
-		(at 76.2 83.82)
 	)
 	(no_connect
@@
 	)
 	(symbol
+		(lib_id "power:GND")
+		(at 76.2 83.82 0)
+		(unit 1)
+		(exclude_from_sim no)
+		(in_bom yes)
+		(on_board yes)
+		(dnp no)
+		(fields_autoplaced yes)
+		(property "Reference" "#PWR062"
+			(at 76.2 90.17 0)
+			(effects
+				(font
+					(size 1.27 1.27)
+				)
+				(hide yes)
+			)
+		)
+		(property "Value" "GND"
+			(at 76.2 88.9 0)
+			(effects
+				(font
+					(size 1.27 1.27)
+				)
+			)
+		)
+		(property "Footprint" ""
+			(at 76.2 83.82 0)
+			(effects
+				(font
+					(size 1.27 1.27)
+				)
+				(hide yes)
+			)
+		)
+		(property "Datasheet" ""
+			(at 76.2 83.82 0)
+			(effects
+				(font
+					(size 1.27 1.27)
+				)
+				(hide yes)
+			)
+		)
+		(property "Description" "Power symbol creates a global label with name \"GND\" , ground"
+			(at 76.2 83.82 0)
+			(effects
+				(font
+					(size 1.27 1.27)
+				)
+				(hide yes)
+			)
+		)
+		(pin "1"
+		)
+		(instances
+			(project "Main"
+				(path "/a34d77bc-8f6a-417e-a206-3165e6c5c658/1fa8e4ec-3b8f-41b7-8956-25ba2b294586"
+					(reference "#PWR062")
+					(unit 1)
+				)
+			)
+		)
+	)
+	(symbol
 		(lib_id "power:+5V")
 		(at 193.04 68.58 0)
@@
 				(path "/a34d77bc-8f6a-417e-a206-3165e6c5c658/1fa8e4ec-3b8f-41b7-8956-25ba2b294586"
 					(reference "L1")
+					(unit 1)
+				)
+			)
+		)
+	)
+	(symbol
+		(lib_id "power:GND")
+		(at 53.34 71.12 0)
+		(unit 1)
+		(exclude_from_sim no)
+		(in_bom yes)
+		(on_board yes)
+		(dnp no)
+		(fields_autoplaced yes)
+		(property "Reference" "#PWR065"
+			(at 53.34 77.47 0)
+			(effects
+				(font
+					(size 1.27 1.27)
+				)
+				(hide yes)
+			)
+		)
+		(property "Value" "GND"
+			(at 53.34 76.2 0)
+			(effects
+				(font
+					(size 1.27 1.27)
+				)
+			)
+		)
+		(property "Footprint" ""
+			(at 53.34 71.12 0)
+			(effects
+				(font
+					(size 1.27 1.27)
+				)
+				(hide yes)
+			)
+		)
+		(property "Datasheet" ""
+			(at 53.34 71.12 0)
+			(effects
+				(font
+					(size 1.27 1.27)
+				)
+				(hide yes)
+			)
+		)
+		(property "Description" "Power symbol creates a global label with name \"GND\" , ground"
+			(at 53.34 71.12 0)
+			(effects
+				(font
+					(size 1.27 1.27)
+				)
+				(hide yes)
+			)
+		)
+		(pin "1"
+		)
+		(instances
+			(project "Main"
+				(path "/a34d77bc-8f6a-417e-a206-3165e6c5c658/1fa8e4ec-3b8f-41b7-8956-25ba2b294586"
+					(reference "#PWR065")
 					(unit 1)
 				)
@@
 					(unit 1)
 				)
+			)
+		)
+	)
+	(symbol
+		(lib_id "power:GND")
+		(at 53.34 73.66 0)
+		(unit 1)
+		(exclude_from_sim no)
+		(in_bom yes)
+		(on_board yes)
+		(dnp no)
+		(fields_autoplaced yes)
+		(property "Reference" "#PWR064"
+			(at 53.34 80.01 0)
+			(effects
+				(font
+					(size 1.27 1.27)
+				)
+				(hide yes)
+			)
+		)
+		(property "Value" "GND"
+			(at 53.34 78.74 0)
+			(effects
+				(font
+					(size 1.27 1.27)
+				)
+			)
+		)
+		(property "Footprint" ""
+			(at 53.34 73.66 0)
+			(effects
+				(font
+					(size 1.27 1.27)
+				)
+				(hide yes)
+			)
+		)
+		(property "Datasheet" ""
+			(at 53.34 73.66 0)
+			(effects
+				(font
+					(size 1.27 1.27)
+				)
+				(hide yes)
+			)
+		)
+		(property "Description" "Power symbol creates a global label with name \"GND\" , ground"
+			(at 53.34 73.66 0)
+			(effects
+				(font
+					(size 1.27 1.27)
+				)
+				(hide yes)
+			)
+		)
+		(pin "1"
+		)
+		(instances
+			(project "Main"
+				(path "/a34d77bc-8f6a-417e-a206-3165e6c5c658/1fa8e4ec-3b8f-41b7-8956-25ba2b294586"
+					(reference "#PWR064")
+					(unit 1)
+				)

Commit message: footprints
Parts:
- L1: footprint LoadCellFootprints:inductor -> Inductor_SMD:L_0805_2012Metric
Changed lines of the file:
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@@
 			)
 		)
-		(property "Footprint" "LoadCellFootprints:inductor"
+		(property "Footprint" "Inductor_SMD:L_0805_2012Metric"
 			(at 124.46 71.12 0)
 			(effects

Commit message: 6 errors
Parts:
- C3, C4, C6, C8, C9: footprint LoadCellFootprints:0p1uF -> Capacitor_SMD:C_0603_1608Metric
- C5, C7: footprint LoadCellFootprints:10uF -> Capacitor_SMD:C_0603_1608Metric
Changed lines of the file:
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@@
 			)
 		)
-		(property "Footprint" "LoadCellFootprints:10uF"
+		(property "Footprint" "Capacitor_SMD:C_0603_1608Metric"
 			(at 109.22 78.74 0)
 			(effects
@@
 			)
 		)
-		(property "Footprint" "LoadCellFootprints:0p1uF"
+		(property "Footprint" "Capacitor_SMD:C_0603_1608Metric"
 			(at 149.86 101.6 0)
 			(effects
@@
 			)
 		)
-		(property "Footprint" "LoadCellFootprints:0p1uF"
+		(property "Footprint" "Capacitor_SMD:C_0603_1608Metric"
 			(at 92.71 31.75 0)
 			(effects
@@
 			)
 		)
-		(property "Footprint" "LoadCellFootprints:0p1uF"
+		(property "Footprint" "Capacitor_SMD:C_0603_1608Metric"
 			(at 147.32 119.38 0)
 			(effects
@@
 			)
 		)
-		(property "Footprint" "LoadCellFootprints:0p1uF"
+		(property "Footprint" "Capacitor_SMD:C_0603_1608Metric"
 			(at 105.41 31.75 0)
 			(effects
@@
 			)
 		)
-		(property "Footprint" "LoadCellFootprints:0p1uF"
+		(property "Footprint" "Capacitor_SMD:C_0603_1608Metric"
 			(at 99.06 78.74 0)
 			(effects
@@
 			)
 		)
-		(property "Footprint" "LoadCellFootprints:10uF"
+		(property "Footprint" "Capacitor_SMD:C_0603_1608Metric"
 			(at 120.65 31.75 0)
 			(effects

Commit message: footprints
Parts:
- DNP3: footprint LoadCellFootprints:10k -> Resistor_SMD:R_0603_1608Metric
Changed lines of the file:
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@@
 			)
 		)
-		(property "Footprint" "LoadCellFootprints:10k"
+		(property "Footprint" "Resistor_SMD:R_0603_1608Metric"
 			(at 204.978 74.93 90)
 			(effects
